File: keyBOARD/keyboard.kicad_pcb (KiCad board)
At the start: 2 copper layers, 141.2 x 114.2 mm, 52 parts, among them J4 AudioJack4, J5 JT8P-3.2T- -1-16Y, SW1 SW_MEC_5G, SW10 SW_MEC_5G, SW11 SW_MEC_5G, SW12 SW_MEC_5G, SW13 SW_MEC_5G, SW14 SW_MEC_5G, SW15 SW_MEC_5G, SW16 SW_key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

Commit message: i
Routing:
- net GPIO23: track 176.4 -> 179.5 mm
- net GPIO19: track 125.5 -> 128.0 mm
- net GPIO21: track 152.5 -> 153.7 mm
- net GND: vias 34 -> 38
